File: hardware/plinkykeeb2_21Jan2022.sch (EAGLE design)
At the start: 93 parts, among them J1 SJ-3523-SMT, J2 SJ-3523-SMT, SW1 KAILH_SOCKETBOX_JADE, SW10 KAILH_SOCKETBOX_JADE, SW11 KAILH_SOCKETBOX_JADE, SW12 KAILH_SOCKETBOX_JADE, SW13 KAILH_SOCKETBOX_JADE, SW14 KAILH_SOCKETBOX_JADE, SW15 KAILH_SOCKETBOX_JADE, SW16 KAILH_SOCKETBOX_JADE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

Commit message: rejiggered audio out
Connections:
- net N$45 renamed MIDIOUT
- net PWM_AUDIO: now also U1.RXI; no longer U1.11(MOSI)
Changed lines of the file:
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@@
 <text x="129.54" y="110.744" size="1.778" layer="97">From "3.4.1. PWM Audio" of
 "Hardware Design w/ RP2040"</text>
-<text x="190.5" y="110.744" size="1.778" layer="97">PWM AUDIO OUT</text>
-<text x="187.96" y="52.324" size="1.778" layer="97">TRS-A MIDI OUT</text>
+<text x="195.58" y="110.744" size="1.778" layer="97">PWM AUDIO OUT</text>
+<text x="195.58" y="54.864" size="1.778" layer="97">TRS-A MIDI OUT</text>
 </plain>
 <instances>
@@
 </segment>
 </net>
-<net name="N$45" class="0">
+<net name="MIDIOUT" class="0">
 <segment>
 <pinref part="R1" gate="G$1" pin="2"/>
@@
 <wire x1="88.9" y1="160.02" x2="88.9" y2="71.12" width="0.1524" layer="91"/>
 <wire x1="88.9" y1="71.12" x2="175.26" y2="71.12" width="0.1524" layer="91"/>
+<label x="93.98" y="160.02" size="1.778" layer="95"/>
 </segment>
 </net>
@@
 <segment>
 <pinref part="R7" gate="G$1" pin="2"/>
-<wire x1="132.08" y1="101.6" x2="127" y2="101.6" width="0.1524" layer="91"/>
-<wire x1="127" y1="101.6" x2="127" y2="119.38" width="0.1524" layer="91"/>
-<wire x1="127" y1="119.38" x2="149.86" y2="119.38" width="0.1524" layer="91"/>
-<pinref part="U1" gate="G$1" pin="11(MOSI)"/>
-<wire x1="132.08" y1="134.62" x2="149.86" y2="134.62" width="0.1524" layer="91"/>
-<wire x1="149.86" y1="134.62" x2="149.86" y2="119.38" width="0.1524" layer="91"/>
-<label x="137.16" y="134.62" size="1.778" layer="95"/>
-</segment>
-</net>
+<wire x1="132.08" y1="101.6" x2="91.44" y2="101.6" width="0.1524" layer="91"/>
+<label x="93.98" y="157.48" size="1.778" layer="95"/>
+<pinref part="U1" gate="G$1" pin="RXI"/>
+<wire x1="109.22" y1="157.48" x2="91.44" y2="157.48" width="0.1524" layer="91"/>
+<wire x1="91.44" y1="157.48" x2="91.44" y2="101.6" width="0.1524" layer="91"/>
+</segment>
+</net>
