File: hardware/plinkykeeb_21Jan2022.brd (EAGLE design)
At the start: 255.3 x 44.5 mm, 93 parts, among them J1 SJ-3523-SMT, J2 SJ-3523-SMT, SW1 KAILH_SOCKETBOX_JADE, SW10 KAILH_SOCKETBOX_JADE, SW11 KAILH_SOCKETBOX_JADE, SW12 KAILH_SOCKETBOX_JADE, SW13 KAILH_SOCKETBOX_JADE, SW14 KAILH_SOCKETBOX_JADE, SW15 KAILH_SOCKETBOX_JADE, SW16 KAILH_SOCKETBOX_JADE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

Commit message: shrink pcb a bit so parts can be 3dprinted
Parts:
- moved R1 3.47 mm to (241.9, 18.9)
- moved R2 3.47 mm to (241.9, 16.4)
- moved J2 3.47 mm to (245.7, 7.75)
- moved J1 3.47 mm to (245.7, 18.5)
- moved C21 2.36 mm to (240.7, 11.3)
- moved C22 2.36 mm to (243.2, 11.3)
- moved R3 2.36 mm to (233.0, 11.3)
- moved R4 2.36 mm to (235.6, 11.3)
- moved R5 2.36 mm to (238.1, 11.3)
- moved R6 2.36 mm to (245.7, 11.3)
- moved R7 2.36 mm to (248.3, 11.3)
- moved U1 1.55 mm to (232.4, 33.4)
- moved C20 1.27 mm to (224.8, 2.54)
- moved D20 1.27 mm to (224.8, 20.3)
- moved LED20 1.27 mm to (224.8, 6.35)
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Routing:
- net ROW4: track 99.5 -> 96.5 mm
- net GND: track 10.5 -> 13.3 mm
- net COL2: track 273.1 -> 270.9 mm
- net COL5: track 255.4 -> 253.2 mm
- net N$46: track 15.7 -> 17.9 mm
- net COL4: track 216.1 -> 214.1 mm
- net ROW2: track 210.0 -> 208.3 mm
- net ROW3: track 153.5 -> 151.8 mm
- net COL3: track 244.7 -> 243.1 mm
- net COL1: track 268.7 -> 267.1 mm
- net +3V3: track 13.9 -> 15.2 mm
- net N$44: track 11.4 -> 10.2 mm
- net N$38: track 16.9 -> 15.6 mm
- net PWM_AUDIO: track 35.5 -> 36.6 mm
- net NEOPIXEL: track 280.7 -> 279.8 mm
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Other:
- board size 255.3 x 44.5 mm -> 254.1 x 43.2 mm

Commit message: submitted to pcbway
Parts:
- added U$1: (no value), todstuff:PLINKY_KEEB_BG_LOGO3
Other:
- board size 254.1 x 43.2 mm -> 254 x 43.2 mm
- board text removed: ""A""
- board text removed: ""AUDIO""
- board text removed: "KB2040 PRO MICRO"
- board text removed: "MIDIOUT"
- board text removed: "plinkykeeb"
Changed lines of the file:
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@@
 <layer number="14" name="Route14" color="22" fill="1" visible="no" active="no"/>
 <layer number="15" name="Route15" color="23" fill="1" visible="no" active="no"/>
-<layer number="16" name="Bottom" color="1" fill="1" visible="yes" active="yes"/>
+<layer number="16" name="Bottom" color="1" fill="1" visible="no" active="yes"/>
 <layer number="17" name="Pads" color="2" fill="1" visible="yes" active="yes"/>
 <layer number="18" name="Vias" color="2" fill="1" visible="yes" active="yes"/>
@@
 <layer number="20" name="Dimension" color="15" fill="1" visible="yes" active="yes"/>
 <layer number="21" name="tPlace" color="7" fill="1" visible="yes" active="yes"/>
-<layer number="22" name="bPlace" color="7" fill="1" visible="yes" active="yes"/>
+<layer number="22" name="bPlace" color="7" fill="1" visible="no" active="yes"/>
 <layer number="23" name="tOrigins" color="15" fill="1" visible="yes" active="yes"/>
-<layer number="24" name="bOrigins" color="15" fill="1" visible="yes" active="yes"/>
+<layer number="24" name="bOrigins" color="15" fill="1" visible="no" active="yes"/>
 <layer number="25" name="tNames" color="7" fill="1" visible="yes" active="yes"/>
-<layer number="26" name="bNames" color="7" fill="1" visible="yes" active="yes"/>
+<layer number="26" name="bNames" color="7" fill="1" visible="no" active="yes"/>
 <layer number="27" name="tValues" color="7" fill="1" visible="no" active="yes"/>
 <layer number="28" name="bValues" color="7" fill="1" visible="no" active="yes"/>
@@
 <layer number="38" name="bTest" color="7" fill="1" visible="no" active="yes"/>
 <layer number="39" name="tKeepout" color="4" fill="11" visible="yes" active="yes"/>
-<layer number="40" name="bKeepout" color="1" fill="11" visible="yes" active="yes"/>
+<layer number="40" name="bKeepout" color="1" fill="11" visible="no" active="yes"/>
 <layer number="41" name="tRestrict" color="4" fill="10" visible="yes" active="yes"/>
-<layer number="42" name="bRestrict" color="1" fill="10" visible="yes" active="yes"/>
+<layer number="42" name="bRestrict" color="1" fill="10" visible="no" active="yes"/>
 <layer number="43" name="vRestrict" color="2" fill="10" visible="no" active="yes"/>
 <layer number="44" name="Drills" color="7" fill="1" visible="no" active="yes"/>
-<layer number="45" name="Holes" color="7" fill="1" visible="yes" active="yes"/>
+<layer number="45" name="Holes" color="7" fill="1" visible="no" active="yes"/>
 <layer number="46" name="Milling" color="3" fill="1" visible="no" active="yes"/>
-<layer number="47" name="Measures" color="7" fill="1" visible="yes" active="yes"/>
-<layer number="48" name="Document" color="7" fill="1" visible="yes" active="yes"/>
-<layer number="49" name="Reference" color="7" fill="1" visible="yes" active="yes"/>
+<layer number="47" name="Measures" color="7" fill="1" visible="no" active="yes"/>
+<layer number="48" name="Document" color="7" fill="1" visible="no" active="yes"/>
+<layer number="49" name="Reference" color="7" fill="1" visible="no" active="yes"/>
 <layer number="50" name="dxf" color="7" fill="1" visible="no" active="no"/>
 <layer number="51" name="tDocu" color="7" fill="1" visible="yes" active="yes"/>
-<layer number="52" name="bDocu" color="7" fill="1" visible="yes" active="yes"/>
+<layer number="52" name="bDocu" color="7" fill="1" visible="no" active="yes"/>
 <layer number="53" name="tGND_GNDA" color="7" fill="9" visible="no" active="no"/>
 <layer number="54" name="bGND_GNDA" color="1" fill="9" visible="no" active="no"/>
@@
 <layer number="114" name="Badge_Outline" color="11" fill="1" visible="no" active="no"/>
 <layer number="115" name="ReferenceISLANDS" color="7" fill="1" visible="no" active="yes"/>
-<layer number="116" name="Patch_BOT" color="9" fill="4" visible="yes" active="yes"/>
+<layer number="116" name="Patch_BOT" color="9" fill="4" visible="no" active="yes"/>
 <layer number="117" name="BACKMAAT1" color="7" fill="1" visible="no" active="yes"/>
 <layer number="118" name="Rect_Pads" color="7" fill="1" visible="no" active="yes"/>
@@
 <layer number="196" name="mValues" color="7" fill="1" visible="no" active="yes"/>
 <layer number="199" name="Contour" color="7" fill="1" visible="no" active="yes"/>
-<layer number="200" name="200bmp" color="1" fill="10" visible="no" active="yes"/>
+<layer number="200" name="200bmp" color="1" fill="10" visible="yes" active="yes"/>
 <layer number="201" name="201bmp" color="2" fill="10" visible="no" active="yes"/>
 <layer number="202" name="202bmp" color="3" fill="10" visible="no" active="yes"/>
@@
 <layer number="205" name="205bmp" color="6" fill="10" visible="no" active="yes"/>
 <layer number="206" name="206bmp" color="7" fill="10" visible="no" active="yes"/>
-<layer number="207" name="207bmp" color="8" fill="10" visible="yes" active="yes"/>
-<layer number="208" name="208bmp" color="9" fill="10" visible="yes" active="yes"/>
-<layer number="209" name="209bmp" color="7" fill="1" visible="yes" active="yes"/>
+<layer number="207" name="207bmp" color="8" fill="10" visible="no" active="yes"/>
+<layer number="208" name="208bmp" color="9" fill="10" visible="no" active="yes"/>
+<layer number="209" name="209bmp" color="7" fill="1" visible="no" active="yes"/>
 <layer number="210" name="210bmp" color="7" fill="1" visible="no" active="yes"/>
 <layer number="211" name="211bmp" color="7" fill="1" visible="no" active="yes"/>
@@
 <wire x1="0" y1="40.64" x2="0" y2="2.54" width="0" layer="20"/>
 <wire x1="0" y1="2.54" x2="2.54" y2="0" width="0" layer="20" curve="90"/>
-<wire x1="2.54" y1="0" x2="252.711109375" y2="0" width="0" layer="20"/>
-<wire x1="252.711109375" y1="0" x2="253.981109375" y2="2.53603125" width="0" layer="20" curve="89.910475"/>
-<wire x1="253.981109375" y1="2.53603125" x2="253.9988875" y2="40.636825" width="0" layer="20"/>
-<wire x1="253.9988875" y1="40.636825" x2="252.7288875" y2="43.18" width="0" layer="20" curve="90.025095"/>
-<wire x1="252.7288875" y1="43.18" x2="2.54" y2="43.18" width="0" layer="20"/>
+<wire x1="2.54" y1="0" x2="251.441665625" y2="0" width="0" layer="20"/>
+<wire x1="251.441665625" y1="0" x2="253.981665625" y2="2.53621875" width="0" layer="20" curve="89.914705"/>
+<wire x1="253.981665625" y1="2.53621875" x2="253.99833125" y2="40.6366375" width="0" layer="20"/>
+<wire x1="253.99833125" y1="40.6366375" x2="251.45833125" y2="43.18" width="0" layer="20" curve="90.025095"/>
+<wire x1="251.45833125" y1="43.18" x2="2.54" y2="43.18" width="0" layer="20"/>
 <wire x1="2.54" y1="43.18" x2="0" y2="40.64" width="0" layer="20" curve="90"/>
 <text x="248.412" y="37.084" size="1.778" layer="22" rot="MR0">KB2040 Pro Micro</text>
@@
 <hole x="60.96" y="30.48" drill="2.54"/>
 <hole x="137.16" y="30.48" drill="2.54"/>
-<hole x="191.77" y="30.48" drill="2.54"/>
-<text x="241.808" y="15.24" size="1.27" layer="21" ratio="10" rot="R180">MIDIOUT</text>
-<text x="241.3" y="4.191" size="1.27" layer="21" ratio="10" rot="R180">"AUDIO"</text>
-<text x="222.377" y="35.433" size="1.778" layer="21" ratio="10">KB2040 PRO MICRO</text>
 <text x="248.412" y="33.274" size="1.778" layer="22" rot="MR0">plinkykeeb2 22Jan2022</text>
 <text x="248.412" y="29.464" size="1.778" layer="22" rot="MR0">github.com/todbot/plinkykeeb</text>
-<text x="249.301" y="15.24" size="1.27" layer="21" ratio="10" rot="R180">"A"</text>
-<text x="3.429" y="22.479" size="1.778" layer="21" ratio="10" rot="R90">plinkykeeb</text>
 </plain>
 <attributes>
@@
 <attribute name="VALUE" x="248.95073125" y="14.35881875" size="1.27228125" layer="27" rot="R180"/>
 </element>
+<element name="U$1" library="todstuff" library_urn="urn:adsk.eagle:library:1731349" package="PLINKY_KEEB_BG_LOGO3" value="" x="0" y="0" smashed="yes"/>
 </elements>
 <signals>

Commit message: docs
Parts:
- moved R2 7.48 mm to (234.9, 19.1), turned to 90 degrees
- moved C22 0.65 mm to (242.6, 11.4)
- moved R4 0.65 mm to (234.9, 11.4)
- moved R1 0.65 mm to (242.6, 19.1), turned to 90 degrees
- moved C21 0.65 mm to (240.0, 11.4)
- moved R3 0.65 mm to (232.4, 11.4)
- moved R5 0.65 mm to (237.5, 11.4)
- moved R6 0.65 mm to (245.1, 11.4)
- moved R7 0.65 mm to (247.7, 11.4)
Routing:
- net +3V3: track 15.2 -> 6.83 mm
- net N$43: track 4.16 -> 11.8 mm
- net N$42: track 6.22 -> 8.48 mm
- net MIDIOUT: track 24.3 -> 23.5 mm
