File: hardware/plinkykeeb_choc_12Feb2022.brd (EAGLE design)
At the start: 250.1 x 43.2 mm, 93 parts, among them J1 SJ-3523-SMT, J2 SJ-3523-SMT, SW1 KBD_SWITCHKALIH_CHOC_SOCKET, SW10 KBD_SWITCHKALIH_CHOC_SOCKET, SW11 KBD_SWITCHKALIH_CHOC_SOCKET, SW12 KBD_SWITCHKALIH_CHOC_SOCKET, SW13 KBD_SWITCHKALIH_CHOC_SOCKET, SW14 KBD_SWITCHKALIH_CHOC_SOCKET, SW15 KBD_SWITCHKALIH_CHOC_SOCKET, SW16 KBD_SWITCHKALIH_CHOC_SOCKET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

Commit message: choc updates
Routing:
- net COL1: track 248.0 -> 247.0 mm
Changed lines of the file:
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@@
 <layer number="196" name="mValues" color="7" fill="1" visible="no" active="yes"/>
 <layer number="199" name="Contour" color="7" fill="1" visible="no" active="yes"/>
-<layer number="200" name="200bmp" color="1" fill="10" visible="no" active="yes"/>
-<layer number="201" name="201bmp" color="2" fill="10" visible="no" active="yes"/>
-<layer number="202" name="202bmp" color="3" fill="10" visible="no" active="yes"/>
+<layer number="200" name="200bmp" color="1" fill="10" visible="yes" active="yes"/>
+<layer number="201" name="201bmp" color="2" fill="10" visible="yes" active="yes"/>
+<layer number="202" name="202bmp" color="3" fill="10" visible="yes" active="yes"/>
 <layer number="203" name="203bmp" color="4" fill="10" visible="no" active="yes"/>
 <layer number="204" name="204bmp" color="5" fill="10" visible="no" active="yes"/>
 <layer number="205" name="205bmp" color="6" fill="10" visible="no" active="yes"/>
 <layer number="206" name="206bmp" color="7" fill="10" visible="no" active="yes"/>
-<layer number="207" name="207bmp" color="8" fill="10" visible="yes" active="yes"/>
+<layer number="207" name="207bmp" color="8" fill="10" visible="no" active="yes"/>
 <layer number="208" name="208bmp" color="9" fill="10" visible="yes" active="yes"/>
 <layer number="209" name="209bmp" color="7" fill="1" visible="yes" active="yes"/>
@@
 </layers>
 <board>
-<fusionsync huburn="a.cGVyc29uYWw6dWUyOWMzMmM3" projecturn="a.cGVyc29uYWw6dWUyOWMzMmM3IzIwMTgwMjExMTE3NDU0Nzgx" f3durn="urn:adsk.wipprod:dm.lineage:4HSctej6Rcm30rx-z4yGEg" pcbguid="" lastpulledtime="" lastsyncedchangeguid="" latestrevisionid="8855fd7d-d5df-4cbd-8284-c39dc488c9be" lastsyncedrevisionid="8855fd7d-d5df-4cbd-8284-c39dc488c9be" lastboardhashguid="5f43b209-c9d0-628b-38e8-ab44c5411fee" lastpushedtime="2022-02-02T01:43:49Z" linktopcb3d="false"/>
+<fusionteam huburn="a.cGVyc29uYWw6dWUyOWMzMmM3" projecturn="a.cGVyc29uYWw6dWUyOWMzMmM3IzIwMTQwNTIyMTMwODUwMQ" folderUrn="urn:adsk.wipprod:fs.folder:co.hppk1xOhTZ6C9BKK3fAJUg" urn="urn:adsk.wipprod:dm.lineage:2vhvDwxjSxC-K6p5w5Q--Q"  versionUrn="urn:adsk.wipprod:fs.file:vf.2vhvDwxjSxC-K6p5w5Q--Q?version=1" camFileUrn="" camFileVersionUrn="" lastpublishedchangeguid="2f74d3c6-43c7-99e9-ae9b-b9cf22c17f74"/>
 <plain>
 <wire x1="0" y1="40.64" x2="0" y2="2.54" width="0" layer="20"/>
@@
 <attribute name="MF" value="CUI Devices" x="245" y="7.62" size="1.778" layer="27" ratio="10" rot="R180" display="off"/>
 <attribute name="MP" value="SJ-3523-SMT-TR" x="245" y="7.62" size="1.778" layer="27" ratio="10" rot="R180" display="off"/>
-<attribute name="NAME" x="249.006309375" y="7.341740625" size="1.27233125" layer="25"/>
+<attribute name="NAME" x="246.506309375" y="7.141740625" size="1.27233125" layer="25"/>
 <attribute name="PACKAGE" value="None" x="245" y="7.62" size="1.778" layer="27" ratio="10" rot="R180" display="off"/>
 <attribute name="PURCHASE-URL" value="https://pricing.snapeda.com/search/part/SJ-3523-SMT-TR/?ref=eda" x="245" y="7.62" size="1.778" layer="27" ratio="10" rot="R180" display="off"/>
@@
 <attribute name="MF" value="CUI Devices" x="245" y="18.542" size="1.778" layer="27" ratio="10" rot="R180" display="off"/>
 <attribute name="MP" value="SJ-3523-SMT-TR" x="245" y="18.542" size="1.778" layer="27" ratio="10" rot="R180" display="off"/>
-<attribute name="NAME" x="248.752309375" y="18.263740625" size="1.27233125" layer="25"/>
+<attribute name="NAME" x="246.452309375" y="18.063740625" size="1.27233125" layer="25"/>
 <attribute name="PACKAGE" value="None" x="245" y="18.542" size="1.778" layer="27" ratio="10" rot="R180" display="off"/>
 <attribute name="PURCHASE-URL" value="https://pricing.snapeda.com/search/part/SJ-3523-SMT-TR/?ref=eda" x="245" y="18.542" size="1.778" layer="27" ratio="10" rot="R180" display="off"/>
@@
 <wire x1="109.3932" y1="37" x2="109.4" y2="37" width="0.2032" layer="16"/>
 <via x="109.4" y="37" extent="1-16" drill="0.4064"/>
-<wire x1="109.4" y1="37" x2="82" y2="37" width="0.2032" layer="1"/>
-<wire x1="76.5" y1="31.5" x2="68.6" y2="31.5" width="0.2032" layer="1"/>
-<wire x1="68.6" y1="31.5" x2="64.5" y2="27.4" width="0.2032" layer="1"/>
-<wire x1="64.5" y1="27.4" x2="64.5" y2="23.2" width="0.2032" layer="1"/>
-<wire x1="82" y1="37" x2="76.5" y2="31.5" width="0.2032" layer="1"/>
+<wire x1="109.4" y1="37" x2="75.8" y2="37" width="0.2032" layer="1"/>
+<wire x1="75.8" y1="37" x2="64.5" y2="25.7" width="0.2032" layer="1"/>
+<wire x1="64.5" y1="25.7" x2="64.5" y2="23.2" width="0.2032" layer="1"/>
 <wire x1="163.4" y1="36.9" x2="163.3" y2="37" width="0.2032" layer="1"/>
 <wire x1="163.3" y1="37" x2="109.4" y2="37" width="0.2032" layer="1"/>
@@
 <wire x1="162" y1="18.2442125" x2="162" y2="21.4" width="0.2032" layer="16"/>
 <wire x1="161.1244" y1="10.6291875" x2="161.1244" y2="17.3686125" width="0.2032" layer="16"/>
-<wire x1="162" y1="21.4" x2="160.4" y2="23" width="0.2032" layer="1"/>
-<wire x1="160.4" y1="23" x2="157.5" y2="23" width="0.2032" layer="1"/>
-<wire x1="166.5" y1="5.5" x2="168.5" y2="5.5" width="0.2032" layer="1"/>
-<wire x1="168.5" y1="5.5" x2="169.8" y2="4.2" width="0.2032" layer="1"/>
-<wire x1="169.8" y1="4.2" x2="218.2" y2="4.2" width="0.2032" layer="1"/>
+<wire x1="162" y1="21.4" x2="159" y2="21.4" width="0.2032" layer="1"/>
+<wire x1="157.5" y1="23" x2="157.5" y2="22.9" width="0.2032" layer="1"/>
+<wire x1="159" y1="21.4" x2="157.5" y2="22.9" width="0.2032" layer="1"/>
+<wire x1="166.5" y1="5.5" x2="167.8" y2="4.2" width="0.2032" layer="1"/>
+<wire x1="167.8" y1="4.2" x2="218.2" y2="4.2" width="0.2032" layer="1"/>
 <via x="218.2" y="4.2" extent="1-16" drill="0.4064"/>
 <wire x1="218.2" y1="4.2" x2="218.2" y2="6.68105" width="0.2032" layer="16"/>
@@
 </signals>
 <mfgpreviewcolors>
-<mfgpreviewcolor name="soldermaskcolor" color="0xC8FFFFFF"/>
-<mfgpreviewcolor name="silkscreencolor" color="0xFF000000"/>
+<mfgpreviewcolor name="soldermaskcolor" color="0xC8000000"/>
+<mfgpreviewcolor name="silkscreencolor" color="0xFFFFFFFF"/>
 <mfgpreviewcolor name="backgroundcolor" color="0xFF282828"/>
 <mfgpreviewcolor name="coppercolor" color="0xFFFFBF00"/>
@@
 </note>
 <note version="8.3" severity="warning">
-Since Version 8.3, EAGLE supports Fusion synchronisation.
-This feature will not be available in this version and saving
-the document will break the link to the Fusion PCB feature.
-</note>
-<note version="8.3" severity="warning">

Commit message: choc updates
Parts:
- moved R1 29.1 mm to (243.0, 28.5), turned to 0 degrees
- moved R2 29.1 mm to (243.0, 31.0), turned to 0 degrees
- moved J2 1.83 mm to (243.5, 17.5)
- moved J1 1.50 mm to (244.0, 6.50)
- moved C21 1.12 mm to (229.0, 14.5)
- moved C22 1.12 mm to (229.0, 17.0)
- moved R3 1.12 mm to (229.0, 7.00)
- moved R4 1.12 mm to (229.0, 9.50)
- moved R5 1.12 mm to (229.0, 12.0)
- moved R6 1.12 mm to (229.0, 19.5)
- moved R7 1.12 mm to (229.0, 22.0)
- moved U1 0.91 mm to (228.0, 32.0), flipped to the top, turned to 270 degrees
Routing:
- net +3V3: track 59.4 -> 11.5 mm, vias 0 -> 1
- net PWM_AUDIO: track 9.84 -> 33.0 mm
- net ROW3: track 166.0 -> 186.3 mm, vias 7 -> 9
- net N$42: track 14.4 -> 30.4 mm, vias 1 -> 3
- net MIDIOUT: track 25.1 -> 9.18 mm
- net COL5: track 187.0 -> 202.1 mm, vias 4 -> 5
- net N$43: track 18.7 -> 33.6 mm
- net ROW1: track 273.4 -> 287.8 mm
- net ROW2: track 217.8 -> 231.8 mm
- net ROW4: track 116.1 -> 105.7 mm
- net NEOPIXEL: track 250.1 -> 260.3 mm
- net COL3: track 218.5 -> 226.7 mm, vias 6 -> 5
- net COL4: track 213.2 -> 205.7 mm, vias 5 -> 4
- net COL2: track 267.5 -> 261.9 mm, vias 5 -> 4
- net COL1: track 247.0 -> 243.5 mm
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Other:
- board size 250.1 x 43.2 mm -> 250 x 43.2 mm

Commit message: plinkykeeb_choc_12Feb sent to fab
Parts:
- moved J1 1.50 mm to (244.0, 8.00)
- moved J2 1.39 mm to (244.0, 18.8)
- moved U1 1.00 mm to (228.0, 33.0)
Routing:
- net N$43: track 33.6 -> 31.9 mm
- net N$42: track 30.4 -> 28.6 mm
- net N$44: track 20.3 -> 21.8 mm
- net N$46: track 19.4 -> 20.5 mm
- net ROW3: track 186.3 -> 187.3 mm
- net ROW2: track 231.8 -> 232.8 mm
- net ROW1: track 287.8 -> 288.8 mm
- net MIDIOUT: track 9.18 -> 10.2 mm
- net COL5: track 202.1 -> 203.1 mm
- net COL4: track 205.7 -> 206.7 mm
- net COL3: track 226.7 -> 227.7 mm
- net COL2: track 261.9 -> 262.9 mm
- net COL1: track 243.5 -> 244.5 mm
- net +3V3: track 11.5 -> 10.5 mm
- net PWM_AUDIO: track 33.0 -> 34.0 mm
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Other:
- board text added: "/Users/tod/projects/synth/plinkykeeb/hardware/fooD.bmp"
